File: Hardware/SpaceCenter_TouchBoard_KiCAD_Rev2/SpaceCenter_TouchBoard_KiCAD.kicad_pcb (KiCad board)
At the start: 2 copper layers, 19.5 x 21 mm, 15 parts, among them J1 Conn_01x05_Male, J2 TOUCH_SENSOR, U1 MTCH101T-I_OT

Commit message: Touch Board rev 2.0 Working Great
Parts:
- R2: value 100k -> 200k
