File: Hardware/SpaceCenter_TouchBoard_KiCAD_Rev2/SpaceCenter_TouchBoard_KiCAD.sch (KiCad schematic (older format))
At the start: 15 parts, among them J1 Conn_01x05_Male, J2 TOUCH_SENSOR, U1 MTCH101T-I_OT

Commit message: Touch Board rev 2.0 Working Great
Parts:
- R2: value 100k -> 200k
Changed lines of the file:
@@
 P 4810 4220
 F 0 "R2" H 4740 4174 50  0000 R CNN
-F 1 "100k" H 4740 4265 50  0000 R CNN
+F 1 "200k" H 4740 4265 50  0000 R CNN
 F 2 "Resistor_SMD:R_0402_1005Metric_Pad0.72x0.64mm_HandSolder" V 4740 4220 50  0001 C CNN
 F 3 "~" H 4810 4220 50  0001 C CNN
