File: Hardware/SpaceCenter_MainBoard_KiCAD/SpaceCenter_MainBoard_KiCAD.kicad_pcb (KiCad board)
At the start: 2 copper layers, 128 x 90 mm, 117 parts, among them J1 Barrel_Jack_Switch, J10 Conn_01x05_Male, J11 Conn_01x05_Male, J12 Conn_01x05_Male, J13 Conn_01x05_Male, J14 Conn_01x05_Male, J15 Conn_01x05_Male, J16 Conn_01x05_Male, J17 Conn_01x05_Male, J18 Conn_01x05_Male, J19 Conn_01x05_Male, J2 Conn_ARM_JTAG_SWD_10, J20 Conn_01x05_Male, J21 Conn_01x05_Male, J22 Conn_01x05_Male, J23 Conn_01x05_Male, J24 Conn_01x05_Male, J25 Conn_01x05_Male, J26 Conn_01x05_Male, J27 Conn_01x05_Male, J28 Conn_01x05_Male, J29 Conn_01x05_Male, J3 Micro_SD_Card_Det_Hirose_DM3AT, J30 Conn_01x05_Male, J31 Conn_01x05_Male, J32 Conn_01x05_Male, J33 Conn_01x05_Male, J34 Conn_01x05_Male, J35 Conn_01x05_Male, J36 Conn_01x05_Male, J37 Conn_01x05_Male, J38 Conn_01x05_Male, J39 Conn_01x05_Male, J4 Screw_Terminal_01x02, J40 Conn_01x05_Male, J41 Conn_01x05_Male, J42 Conn_01x02_Male, J5 Screw_Terminal_01x02, J6 Conn_01x05_Male, J7 Conn_01x05_Male, J8 Conn_01x05_Male, J9 Conn_01x05_Male, Q1 DMG1012T-7, Q2 DMG1012T-7, U1 MIC5205-3.3YM5, U2 STM32L072VBTx, U3 MAX98357, U4 MAX98357, U5 SN74LVC2T45DCUR, U6 SN74LVC2T45DCUR

Commit message: Picking this project up again
Unsure what the changes are...
Other:
- net class Default removed
