File: Hardware/SpaceCenter_TouchBoard_KiCAD_Rev3/SpaceCenter_TouchBoard_KiCAD.kicad_pcb (KiCad board)
At the start: 2 copper layers, 19.5 x 21 mm, 15 parts, among them J1 Conn_01x05_Male, J2 TOUCH_SENSOR, U1 MTCH101T-I_OT

Commit message: KiCAD Updates
Parts:
- removed R5: DNP, Resistor_SMD:R_0402_1005Metric_Pad0.72x0.64mm_HandSolder
- removed R6: 4.7k, Resistor_SMD:R_0402_1005Metric_Pad0.72x0.64mm_HandSolder
- added C4: 20n, Capacitor_SMD:C_0402_1005Metric_Pad0.74x0.62mm_HandSolder, F.Cu at (129.9, 98.6)
- added C5: 10u, Capacitor_SMD:C_0402_1005Metric_Pad0.74x0.62mm_HandSolder, F.Cu at (144.8, 87.7)
- R1: value 4.7k -> 100k; moved to F.Cu
- R2: value 200k -> 10k
- R3: value 100k -> 1k
- R4: value 4.7k -> 1k
- R7: value 6.8k -> 16.9k
- U1: value MTCH101T-I_OT -> AT42QT1010-TSHR; footprint footprints:MTCH101T-I&slash_OT -> footprints:SOT95P270X145-6N
- moved R7 20.6 mm to (129.9, 90.6), turned to -90 degrees
- moved R1 5.77 mm to (129.9, 96.0)
- moved R3 4.33 mm to (128.6, 93.1)
- moved R2 4.19 mm to (129.9, 93.2), turned to -90 degrees
- moved R4 3.48 mm to (128.6, 90.6)
- moved C3 0.30 mm to (129.2, 100.7)
Connections:
- R1 pad 1: Net-(R1-Pad1) -> Net-(U1-SNSK)
- R2 pad 1: Net-(R2-Pad1) -> CAP_TOUCH
- R2 pad 2: +5V -> Net-(U1-OUT)
- R3 pad 1: GND -> Net-(U1-SYNC)
- R3 pad 2: Net-(R2-Pad1) -> +5V
- R4 pad 1: Net-(R4-Pad1) -> GND
- R4 pad 2: +5V -> Net-(U1-SYNC)
- U1 pad 1: Net-(R1-Pad1) -> Net-(U1-OUT)
- U1 pad 3: Net-(R2-Pad1) -> Net-(U1-SNSK)
- U1 pad 4: CAP_TOUCH -> Net-(U1-SNS)
- U1 pad 6: Net-(R4-Pad1) -> Net-(U1-SYNC)
Routing:
- net Net-(U1-OUT): track 0.00 -> 13.7 mm, vias 0 -> 2
- net Net-(U1-SYNC): track 0.00 -> 12.9 mm
- net Net-(R2-Pad1): track 12.9 -> 0.00 mm, vias 2 -> 0
- net Net-(U1-SNSK): track 0.00 -> 12.2 mm, vias 0 -> 2
- net Net-(R4-Pad1): track 11.5 -> 0.00 mm
- net +5V: track 61.0 -> 52.3 mm
- net Net-(R1-Pad1): track 7.71 -> 0.00 mm, vias 1 -> 0
- net Net-(J2-Pin_1): track 1.25 -> 7.79 mm, vias 1 -> 0
- net Net-(U1-SNS): track 0.00 -> 3.87 mm
- net GND: track 67.3 -> 65.1 mm, vias 6 -> 4
- net CAP_TOUCH: track 24.0 -> 24.1 mm, vias 1 -> 3
Other:
- net class Default removed
- net class Power removed
- board text added: "Touch Board 3.0 AC"
- board text removed: "Touch Board 2.0 AC"
