File: Hardware/SpaceCenter_TouchBoard_KiCAD_Rev3/_autosave-SpaceCenter_TouchBoard_KiCAD.kicad_sch (KiCad schematic)
At the start: 15 parts, among them J1 Conn_01x05_Male, J2 TOUCH_SENSOR, U1 AT42QT1010-TSHR

Commit message: KiCAD Updates
Parts:
- R3: now not fitted
Changed lines of the file:
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@@
   )
   (symbol (lib_id "Device:R") (at 125.984 125.73 0) (mirror x) (unit 1)
-    (in_bom yes) (on_board yes) (dnp no)
+    (in_bom yes) (on_board yes) (dnp yes)
     (property "Reference" "R3" (at 130.048 124.206 0)
       (effects (font (size 1.27 1.27)) (justify right))
